File: PCB/Single.kicad_pcb (KiCad board)
At the start: 2 copper layers, 320.4 x 143.3 mm, 132 parts, among them SW1 SW_Push, SW10 SW_Push, SW11 SW_Push, SW12 SW_Push, SW13 SW_Push, SW14 SW_Push, SW15 SW_Push, SW16 SW_Push, SW17 SW_Push, SW18 SW_Push, SW19 SW_Push, SW2 SW_Push, SW20 SW_Push, SW21 SW_Push, SW22 SW_Push, SW23 SW_Push, SW24 SW_Push, SW25 SW_Push, SW26 SW_Push, SW27 SW_Push, SW28 SW_Push, SW29 SW_Push, SW3 SW_Push, SW30 SW_Push, SW31 SW_Push, SW32 SW_Push, SW33 SW_Push, SW34 SW_Push, SW35 SW_Push, SW36 SW_Push, SW37 SW_Push, SW38 SW_Push, SW39 SW_Push, SW4 SW_Push, SW40 SW_Push, SW41 SW_Push, SW42 SW_Push, SW43 SW_Push, SW44 SW_Push, SW48 SW_Push, SW49 SW_Push, SW5 SW_Push, SW50 SW_Push, SW51 SW_Push, SW52 SW_Push, SW53 SW_Push, SW54 SW_Push, SW55 SW_Push, SW56 SW_Push, SW57 SW_Push, SW58 SW_Push, SW59 SW_Push, SW6 SW_Push, SW60 SW_Push, SW61 SW_Push, SW62 SW_Push, SW63 SW_Push, SW64 SW_Push, SW7 SW_Push, SW8 SW_Push, SW9 SW_Push, U2 MCP23017_SO, U3 XIAO-nRF52840-SMD

Commit message: Added all files required for the display based keyboard
Parts:
- added C2: C2, Capacitor_SMD:C_0805_2012Metric, B.Cu at (131.8, 126.8)
- added C3: C_0402_1005Metric, Capacitor_SMD:C_0402_1005Metric, B.Cu at (131.8, 144.2)
- added Display: MDOB128032GV-WI, Display:MDOB128032GV-WI, F.Cu at (150.8, 136.0)
- added R5: R_0402_1005Metric, Resistor_SMD:R_0402_1005Metric, B.Cu at (60.4, 129.6)
- added REF**: MountingHole_2.2mm_M2_DIN965_Pad_TopBottom, MountingHole:MountingHole_2.2mm_M2_DIN965_Pad_TopBottom, F.Cu at (359.8, 149.3)
- added REF**: MountingHole_2.2mm_M2_DIN965_Pad_TopBottom, MountingHole:MountingHole_2.2mm_M2_DIN965_Pad_TopBottom, F.Cu at (72.5, 260.5)
- added REF**: MountingHole_2.2mm_M2_DIN965_Pad_TopBottom, MountingHole:MountingHole_2.2mm_M2_DIN965_Pad_TopBottom, F.Cu at (201.8, 260.8)
- added REF**: MountingHole_2.2mm_M2_DIN965_Pad_TopBottom, MountingHole:MountingHole_2.2mm_M2_DIN965_Pad_TopBottom, F.Cu at (50.6, 126.5)
- added REF**: MountingHole_2.2mm_M2_DIN965_Pad_TopBottom, MountingHole:MountingHole_2.2mm_M2_DIN965_Pad_TopBottom, F.Cu at (361.3, 261.1)
- C1: value C -> C1; footprint Capacitor_SMD:C_0805_2012Metric -> Capacitor_SMD:C_0603_1608Metric; moved to B.Cu
- R3, R4: moved to B.Cu
- moved Resistor chain1 10.5 mm to (106.0, 142.0), turned to 180 degrees
- moved C1 9.93 mm to (73.1, 127.1)
- moved R4 3.66 mm to (102.4, 130.5)
- moved R3 3.32 mm to (103.1, 126.2)
- moved REF**1 0.05 mm to (92.7, 228.6)
- moved SW44 0.05 mm to (92.8, 228.6)
Connections:
- U2 pad 18: 3V3 -> Reset
Routing:
- net Row 5: track 788.4 -> 546.6 mm, vias 0 -> 2
- net SCL: track 57.9 -> 114.9 mm, vias 2 -> 3
- net GND: track 98.6 -> 153.5 mm, vias 0 -> 1
- net SDA: track 60.5 -> 94.6 mm, vias 4 -> 2
- net Row 2: track 657.3 -> 630.6 mm, vias 3 -> 2
- net Row 3: track 652.0 -> 628.4 mm, vias 4 -> 3
- net Row 1: track 621.2 -> 609.3 mm
- net 3V3: track 173.8 -> 162.1 mm, vias 2 -> 5
- net Row 4: track 431.3 -> 420.4 mm
- net Reset: track 0.00 -> 5.84 mm, vias 0 -> 1
Other:
- board size 320.4 x 143.3 mm -> 317.3 x 143.3 mm

Commit message: Refactor code structure for improved readability and maintainability
Parts:
- added REF**: STAB_MX_6u, PCM_marbastlib-mx:STAB_MX_6u, F.Cu at (202.3, 247.6)
